Commit message: [FEAT] import biped-v3

File: biped_to_unity-v3/biped.urdf (robot description, URDF)
Before this commit: robot biped, 13 links, 12 joints
Links:
- link back_1: mass 0.0027553261785723494 -> 0.005190420000000001
- link base_link: mass 0.0007331653384976692 -> 0.00020390182942264898
- link sacrum_1: mass 0.0001318676695997575 -> 0.0022235524932220385
Joints:
- removed joint Revolute 1
- removed joint Revolute 15
- removed joint Revolute 2
- removed joint Slider 14
- added joint Revolute 18: type continuous, parent base_link, child sacrum_1, origin xyz=0.0039 0.0 0.0055 rpy=0 0 0, axis -1.0 0.0 0.0
- added joint Revolute 20: type continuous, parent base_link, child l_hip_1, origin xyz=0.004 0.0045 -0.0025 rpy=0 0 0, axis 1.0 0.0 0.0
- added joint Revolute 21: type continuous, parent base_link, child r_hip_1, origin xyz=0.004 -0.0045 -0.0025 rpy=0 0 0, axis 1.0 0.0 0.0
- added joint Slider 19: type prismatic, parent sacrum_1, child back_1, origin xyz=-0.0019 0.0 0.0015 rpy=0 0 0, axis 0.0 1.0 0.0, limit lower=-0.004 upper=0.004 effort=100 velocity=100
- joint Revolute 13: axis -1.0 0.0 0.0 -> -1.0 0.0 -0.0
- joint Revolute 4: axis 0.0 1.0 0.0 -> 0.0 1.0 -0.0
- joint Revolute 5: axis -0.0 1.0 0.0 -> -0.0 1.0 -0.0
- joint Revolute 7: axis 0.0 1.0 0.0 -> 0.0 1.0 -0.0
